File: Hardware/CPU-001/CPU-001.sch (EAGLE design)
At the start: 73 parts, among them IC1 IS42S16800F-7TL, J1 10144517-042802LF, J2 10144518-041802LF, J3 10144517-042802LF, J4 10144518-041802LF, J6 2X5_0.05_SWD, U1 ATSAMV71Q19B-AABT, U2 ATA6561-GAQW-N, U6 NCV8170AXV330T2G, U7 ATA6561-GAQW-N

Commit message: more work on CPU-001
Parts:
- added C21: 1uF, rcl:C-EUC0603
Connections:
- removed net +3.5V: C1.1, J3.31, J3.33, J3.35, J3.37, J4.31, J4.33, J4.35, J4.37, U6.EN, U6.IN
- removed net CAN2_N: R39.1, U2.CANL
- removed net CAN2_P: R39.2, U2.CANH
- removed net CANRX2: U2.RXD
- removed net CANTX2: U2.TXD
- removed net CAN_N: J1.6, J2.6
- removed net CAN_P: J1.4, J2.4
- removed net CAN_STBY2: U2.STBY
- removed net RFU_3: J1.3, J2.3
- removed net RFU_5: J1.5, J2.5
- removed net RFU_7: J1.7, J2.7
- new net +12V: J3.17, J3.19, J3.21, J3.23, J3.25, J3.27, J3.29, J4.17, J4.19, J4.21, J4.23, J4.25, J4.27, J4.29
- new net CAN0_N: J1.6, J2.6, R26999.1, U7.CANL
- new net CAN0_P: J1.4, J2.4, R26999.2, U7.CANH
- new net CANRX0: U7.RXD
- new net CANTX0: U7.TXD
- new net CAN_STBY0: U7.STBY
- net +3V3: now also C21.1, U$5.VDD
- net +5V: now also C1.1, J3.31, J3.33, J3.35, J3.37, J4.31, J4.33, J4.35, J4.37, U6.EN, U6.IN; no longer J3.17, J3.19, J3.21, J3.23, J3.25, J3.27, J3.29, J4.17, J4.19, J4.21, J4.23, J4.25, J4.27, J4.29
- net CAN1_N: now also J1.5, J2.5, R39.1, U2.CANL; no longer R26999.1, U7.CANL
- net CAN1_P: now also J1.3, J2.3, R39.2, U2.CANH; no longer R26999.2, U7.CANH
- net CANRX1: now also U2.RXD; no longer U7.RXD
- net CANTX1: now also U2.TXD; no longer U7.TXD
- net CAN_STBY1: now also U2.STBY; no longer U7.STBY
- net GND: now also C21.2, U$5.GND, U$5.GND1, U$5.VSS
- net PA25: now also U$5.SCLK
- net PA26: now also U$5.DAT2
- net PA27: now also U$5.CS
- net PA28: now also U$5.DATA_IN
- net PA30: now also U$5.DATA_OUT
- net PA31: now also U$5.DAT1
- net SHIELD: now also J1.7, J2.7
Other:
- note added: "CAN_STBY0"
- note added: "CAN_STBY1"
- note added: "MCCDA"
- note added: "MCCK"
- note added: "MCDA0"
- note added: "MCDA1"
- note added: "MCDA2"
- note added: "MCDA3"
- moved on the sheet: R89999

Commit message: added altimeter.. working through schematic slowly...
Parts:
- removed U6: NCV8170AXV330T2G, SamacSys_Parts:NCV8170AXV330T2G
- added C20: 1u, rcl:C-EUC0402
- added C22: 100n, rcl:C-EUC0402
- added C23, C24: 10uF, SparkFun-Capacitors:10UF-POLAR-0603-6.3V-20%(TANT)
- added C25, C28: 100nF, rcl:C-EUC0402
- added C26, C27: 1uF, rcl:C-EUC0402
- added IC2: NCV1117ST33T3G, v-reg:LD117ASTR
- added IC3: TLV71318PQDBVRQ1, SamacSys_Parts:NCP718BSN180T1G
- added L1, L2: 470@100MHz, SparkFun-Coils:INDUCTOR-0603-33NH
- added R40, R43, R44: (no value), rcl:R-US_R0402
- added R41, R42: 10k, rcl:R-US_R0402
- added R45: 200k, rcl:R-US_R0402
- added U3: ICP-10111, ICP-10111:ICP-10111
- added U4: PCA9306, SparkFun-IC-Comms:PCA9306PCA9306DC-1:1
- C15, C16: value 100n -> 4.7u; device rcl:C-EUC0402 -> rcl:C-EUC0805
- C21: value 1uF -> 4.7u; device rcl:C-EUC0603 -> rcl:C-EUC0805
- C8: value 10u -> 4.7u
Connections:
- removed net CANRX0: U7.RXD
- removed net CANRX1: U2.RXD
- removed net CANTX0: U7.TXD
- removed net CANTX1: U2.TXD
- removed net CAN_STBY0: U7.STBY
- removed net CAN_STBY1: U2.STBY
- removed net N$2: C3.1, C4.1, C5.1, C6.1, C7.1, U1C.VDDCORE, U1C.VDDCORE_2, U1C.VDDCORE_3, U1C.VDDCORE_4, U1C.VDDCORE_5
- removed net N$3: C10.1, C11.1, C12.1, C13.1, C14.1, C15.1, C16.1, C17.1, C8.1, C9.1, U1C.VDDIN, U1C.VDDIO, U1C.VDDIO_2, U1C.VDDIO_3, U1C.VDDIO_4, U1C.VDDIO_5, U1C.VDDPLLUSB, U1C.VDDTUMII
- new net +1.8V: C25.1, C27.1, IC3.NC/ADJ, IC3.OUT, R41.2, R42.2, U3.VDD, U4.VREF1
- new net N$1: C28.1, R45.2, U4.EN, U4.VREF2
- new net N$4: L2.1, R40.2
- new net SCL0_1V8: R42.1, U3.SCL, U4.SCL1
- new net SDA0_1V8: R41.1, U3.SDA, U4.SDA1
- new net VDDOUT: C17.1, C20.1, C22.1, C3.1, C4.1, C5.1, C6.1, C7.1, L1.1, U1C.VDDCORE, U1C.VDDCORE_2, U1C.VDDCORE_3, U1C.VDDCORE_4, U1C.VDDCORE_5, U1C.VDDOUT, U1C.VDDTUMIC
- new net VDDPLL: C15.1, L1.2, U1C.VDDPLL
- new net VDDPLLUSB: C16.1, L2.2, U1C.VDDPLLUSB
- net +3V3: now also C10.1, C11.1, C12.1, C13.1, C14.1, C23.+, C26.1, C8.1, C9.1, IC2.OUT, IC3.EN, IC3.IN, R40.1, R43.2, R44.2, R45.1, U1C.VDDIN, U1C.VDDIO, U1C.VDDIO_2, U1C.VDDIO_3, U1C.VDDIO_4, U1C.VDDIO_5, U1C.VDDTUMII; no longer U6.OUT
- net +5V: now also C24.+, IC2.IN; no longer U6.EN, U6.IN
- net GND: now also C20.2, C22.2, C23.-, C24.-, C25.2, C26.2, C27.2, C28.2, IC2.ADJ, IC3.GND, U3.GND, U3.RESV2, U3.RESV5, U3.RESV6, U4.GND; no longer U6.GND_1, U6.GND_2
- net PA1: now also U7.STBY
- net PA2: now also U2.STBY
- net PA3: now also R43.1, U4.SDA2
- net PA4: now also R44.1, U4.SCL2
- net PB2: now also U7.TXD
- net PB3: now also U7.RXD
- net PC12: now also U2.RXD
- net PC14: now also U2.TXD
Other:
- note added: "SCL0"
- note added: "SDA0"
- note added: "Should we put usb on this board for config and debug?"
- note added: "can this 1A regulator supply enough current?? (w/o getting too hot)"
- note added: "do we want JTAG or SWD?"
- note added: "do we want an tiny cap/battery backup to try and save the 1k backup sdram in the case of a bus brownout during flight? and do we want an RTC?"
- note added: "do we want the card detect pin for anything?"
- note added: "pullup on SWCLK"

Commit message: updates to CPU-001 and DBG-001
Connections:
- net +3V3: now also IC1.VDDQ_1, IC1.VDDQ_2, IC1.VDDQ_3, IC1.VDDQ_4, IC1.VDD_1, IC1.VDD_2, IC1.VDD_3
- net GND: now also IC1.VSSQ_1, IC1.VSSQ_2, IC1.VSSQ_3, IC1.VSSQ_4, IC1.VSS_1, IC1.VSS_2, IC1.VSS_3
Other:
- moved on the sheet: IC1
