File: Hardware/DBG-001/DBG-001.brd (EAGLE design)
At the start: 78.7 x 94 mm, 23 parts, among them J1 10144517-042802LF, J2 10144518-041802LF, J3 10144517-042802LF, J4 10144518-041802LF, J6 2X5_0.05_SWD, U1 ATSAMC21E15A-AUT, U6 NCV8170AXV330T2G, U7 ATA6561-GAQW-N

Commit message: updates to CPU-001 and DBG-001
Parts:
- removed C32: 1uF, rcl:C0805
- added C10, C9: 100nF, rcl:C0402
- added C4: 1uF, rcl:C0805
- added C5, C6, C7, C8: 100nF, rcl:C0805
- added JP10: (no value), pinhead:1X04
- added JP4: SDA, pinhead:1X02
- added JP5: SCL, pinhead:1X02
- added JP6: MISO, pinhead:1X02
- added JP7: MOSI, pinhead:1X02
- added JP8: SCK, pinhead:1X02
- added JP9: (no value), pinhead:2X20
- added R4: 1k, rcl:R0402
- added R5: 120 DNP, rcl:R0402
- added U3: ATA6561-GAQW-N, SamacSys Managed:SOIC127P600X175-8N
- JP2: value (none) -> SCK; device pinhead:1X01 -> pinhead:1X02
- JP3: device pinhead:1X02 -> pinhead:1X03
- U1: value ATSAMC21E15A-AUT -> ATSAMC21G17A-AUT; device SamacSys_Parts:QFP80P900X900X120-32N -> ATSAM:QFP50P900X900X120-48N
- moved JP3 75.8 mm to (-12.7, -55.9)
- moved U1 50.8 mm to (0.25, -43.7), flipped to the top
- moved JP2 5.01 mm to (25.4, -3.30)
- moved JP1 0.05 mm to (-38.1, -21.8)
- renumbered U7 to U2
Connections:
- net CAN_N renamed CAN0_N
- net CAN_P renamed CAN0_P
- removed net CAN2_N: J1.5, J2.5
- removed net CAN2_P: J1.3, J2.3
- removed net CANRX: U1.24, U2.4
- removed net CANTX: U1.23, U2.1
- removed net CAN_STBY: U1.25, U2.8
- removed net RFU_3: JP1.3
- removed net RFU_5: JP1.5
- removed net RFU_7: JP1.7
- new net CAN0RX: JP9.26, U1.34, U2.4
- new net CAN0TX: JP9.25, U1.33, U2.1
- new net CAN0_STBY: JP9.27, U1.39, U2.8
- new net CAN1RX: JP9.34, U1.20, U3.4
- new net CAN1TX: JP9.33, U1.19, U3.1
- new net CAN1_N: J1.5, J2.5, JP1.5, R5.1, U3.6
- new net CAN1_P: J1.3, J2.3, JP1.3, R5.2, U3.7
- new net CAN1_STBY: JP9.28, U1.41, U3.8
- new net I2C_SCL_R: JP5.1, JP9.18, U1.26
- new net I2C_SDA_R: JP4.1, JP9.17, U1.25
- new net N$1: C4.1, C5.1, U1.43
- new net PA02: JP9.3, U1.3
- new net PA03: JP9.4, U1.4
- new net PA07: JP9.8, U1.12
- new net PA09: JP9.10, U1.14
- new net PA12: JP9.13, U1.21
- new net PA13: JP9.14, U1.22
- new net PA14: JP9.15, U1.23
- new net PA15: JP9.16, U1.24
- new net PA18: JP9.19, U1.27
- new net PA19: JP9.20, U1.28
- new net PA20: JP9.21, U1.29
- new net PA21: JP9.22, U1.30
- new net PA22: JP9.23, U1.31
- new net PA23: JP9.24, U1.32
- new net PB02: JP9.29, U1.47
- new net PB03: JP9.30, U1.48
- new net PB08: JP9.31, U1.7
- new net PB09: JP9.32, U1.8
- new net PB22: JP9.35, U1.37
- new net PB23: JP9.36, U1.38
- new net P_GOOD_R: JP2.1, JP9.7, U1.11
- new net SPI_MISO_R: JP10.1, JP6.1, JP9.9, U1.13
- new net SPI_MOSI_R: JP10.2, JP7.1, JP9.11, U1.15
- new net SPI_SCK_R: JP10.3, JP8.1, JP9.12, U1.16
- net +3V3: now also C10.1, C6.1, C7.1, C8.1, JP9.37, R4.2, U1.17, U1.36, U1.44, U1.6, U3.5; no longer C32.1, U1.29, U1.30, U1.9
- net +5V: now also C9.1, JP9.38, U3.3
- net DETECT_A: now also JP9.1
- net DETECT_B: now also JP9.2
- net GND: now also C10.2, C4.2, C5.2, C6.2, C7.2, C8.2, C9.2, JP1.7, JP10.4, JP3.3, JP9.39, JP9.40, U1.18, U1.35, U1.42, U1.5, U3.2; no longer C32.2, U1.10, U1.28
- net I2C_SCL: now also JP5.2; no longer U1.18
- net I2C_SDA: now also JP4.2; no longer U1.17
- net P_GOOD: now also JP2.2; no longer JP2.1, U1.15
- net RESET: now also U1.40; no longer U1.26
- net SPI_MISO: now also JP6.2; no longer U1.11
- net SPI_MOSI: now also JP7.2; no longer U1.13
- net SPI_SCK: now also JP8.2; no longer U1.14
- net SWCLK: now also R4.1, U1.45; no longer U1.31
- net SWDIO: now also U1.46; no longer U1.32
- net UART_RX: now also JP9.6, U1.10; no longer U1.22
- net UART_TX: now also JP9.5, U1.9; no longer U1.21
Routing:
- net CAN1TX: track 0.00 -> 144.2 mm, vias 0 -> 5
- net CAN1RX: track 0.00 -> 144.2 mm, vias 0 -> 5
- net DETECT_A: track 57.3 -> 190.9 mm, vias 1 -> 2
- net CAN0RX: track 0.00 -> 131.4 mm, vias 0 -> 2
- net CAN0_STBY: track 0.00 -> 121.8 mm, vias 0 -> 3
- net I2C_SDA_R: track 0.00 -> 119.9 mm, vias 0 -> 5
- net +3V3: track 207.2 -> 317.0 mm, vias 5 -> 8
- net DETECT_B: track 22.7 -> 126.4 mm, vias 2 -> 5
- net UART_RX: track 33.3 -> 136.7 mm
- net CAN1_STBY: track 0.00 -> 94.5 mm, vias 0 -> 5
- net CAN0TX: track 0.00 -> 94.2 mm, vias 0 -> 4
- net CAN1_P: track 0.00 -> 93.9 mm, vias 0 -> 5
- net CAN1_N: track 0.00 -> 93.3 mm, vias 0 -> 5
- net SPI_MISO_R: track 0.00 -> 91.7 mm, vias 0 -> 2
- net PA09: track 0.00 -> 84.0 mm, vias 0 -> 4
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Other:
- board size 78.7 x 94 mm -> 86.4 x 94 mm
