File: Hardware/DBG-001/DBG-001.sch (EAGLE design)
At the start: 23 parts, among them J1 10144517-042802LF, J2 10144518-041802LF, J3 10144517-042802LF, J4 10144518-041802LF, J6 2X5_0.05_SWD, U1 ATSAMC21E15A-AUT, U6 NCV8170AXV330T2G, U7 ATA6561-GAQW-N

Commit message: updates to CPU-001 and DBG-001
Parts:
- removed C32: 1uF, rcl:C-EUC0805
- removed U7: ATA6561-GAQW-N, SamacSys Managed:ATA6561-GAQW-N
- added C10, C9: 100nF, rcl:C-EUC0402
- added C4: 1uF, rcl:C-EUC0805
- added C5, C6, C7, C8: 100nF, rcl:C-EUC0805
- added JP10: (no value), pinhead:PINHD-1X4
- added JP4: SDA, pinhead:PINHD-1X2
- added JP5: SCL, pinhead:PINHD-1X2
- added JP6: MISO, pinhead:PINHD-1X2
- added JP7: MOSI, pinhead:PINHD-1X2
- added JP8: SCK, pinhead:PINHD-1X2
- added JP9: (no value), pinhead:PINHD-2X20
- added R4: 1k, rcl:R-US_R0402
- added R5: 120 DNP, rcl:R-US_R0402
- added U2, U3: ATA6561-GAQW-N, SamacSys Managed:ATA6561-GAQW-N
- JP2: value (none) -> SCK; device pinhead:PINHD-1X1 -> pinhead:PINHD-1X2
- JP3: device pinhead:PINHD-1X2 -> pinhead:PINHD-1X3
- U1: value ATSAMC21E15A-AUT -> ATSAMC21G17A-AUT; device SamacSys_Parts:ATSAMC21E15A-AUT -> ATSAM:ATSAMC21G17A-AUT
Connections:
- removed net CAN2_N: J1.5, J2.5
- removed net CAN2_P: J1.3, J2.3
- removed net CANRX: U1A.PA25/SERCOM3/PAD3/CAN0RX, U7.RXD
- removed net CANTX: U1A.PA24/SERCOM3/PAD2/CAN0TX, U7.TXD
- removed net CAN_N: J1.6, J2.6, JP1.6, R26.1, U7.CANL
- removed net CAN_P: J1.4, J2.4, JP1.4, R26.2, U7.CANH
- removed net CAN_STBY: U1A.PA27, U7.STBY
- removed net RFU_3: JP1.3
- removed net RFU_5: JP1.5
- removed net RFU_7: JP1.7
- new net CAN0RX: JP9.26, U1G$2.PA25, U2.RXD
- new net CAN0TX: JP9.25, U1G$2.PA24, U2.TXD
- new net CAN0_N: J1.6, J2.6, JP1.6, R26.1, U2.CANL
- new net CAN0_P: J1.4, J2.4, JP1.4, R26.2, U2.CANH
- new net CAN0_STBY: JP9.27, U1G$2.PA27, U2.STBY
- new net CAN1RX: JP9.34, U1G$2.PB11, U3.RXD
- new net CAN1TX: JP9.33, U1G$2.PB10, U3.TXD
- new net CAN1_N: J1.5, J2.5, JP1.5, R5.1, U3.CANL
- new net CAN1_P: J1.3, J2.3, JP1.3, R5.2, U3.CANH
- new net CAN1_STBY: JP9.28, U1G$2.PA28, U3.STBY
- new net I2C_SCL_R: JP5.1, JP9.18, U1G$2.PA17
- new net I2C_SDA_R: JP4.1, JP9.17, U1G$2.PA16
- new net N$1: C4.1, C5.1, U1G$1.VDDCORE
- new net PA02: JP9.3, U1G$2.PA02
- new net PA03: JP9.4, U1G$2.PA03
- new net PA07: JP9.8, U1G$2.PA07
- new net PA09: JP9.10, U1G$2.PA09
- new net PA12: JP9.13, U1G$2.PA12
- new net PA13: JP9.14, U1G$2.PA13
- new net PA14: JP9.15, U1G$2.PA14
- new net PA15: JP9.16, U1G$2.PA15
- new net PA18: JP9.19, U1G$2.PA18
- new net PA19: JP9.20, U1G$2.PA19
- new net PA20: JP9.21, U1G$2.PA20
- new net PA21: JP9.22, U1G$2.PA21
- new net PA22: JP9.23, U1G$2.PA22
- new net PA23: JP9.24, U1G$2.PA23
- new net PB02: JP9.29, U1G$2.PB02
- new net PB03: JP9.30, U1G$2.PB03
- new net PB08: JP9.31, U1G$2.PB08
- new net PB09: JP9.32, U1G$2.PB09
- new net PB22: JP9.35, U1G$2.PB22
- new net PB23: JP9.36, U1G$2.PB23
- new net P_GOOD_R: JP2.1, JP9.7, U1G$2.PA06
- new net SPI_MISO_R: JP10.1, JP6.1, JP9.9, U1G$2.PA08
- new net SPI_MOSI_R: JP10.2, JP7.1, JP9.11, U1G$2.PA10
- new net SPI_SCK_R: JP10.3, JP8.1, JP9.12, U1G$2.PA11
- net +3V3: now also C10.1, C6.1, C7.1, C8.1, JP9.37, R4.2, U1G$1.VDDANA, U1G$1.VDDIN, U1G$1.VDDIO_1, U1G$1.VDDIO_2, U2.VIO, U3.VIO; no longer C32.1, U1B.VDDANA, U1B.VDDCORE, U1B.VDDIN, U7.VIO
- net +5V: now also C9.1, JP9.38, U2.VCC, U3.VCC; no longer U7.VCC
- net DETECT_A: now also JP9.1, U1G$2.PA00; no longer U1A.PA00
- net DETECT_B: now also JP9.2, U1G$2.PA01; no longer U1A.PA01
- net GND: now also C10.2, C4.2, C5.2, C6.2, C7.2, C8.2, C9.2, JP1.7, JP10.4, JP3.3, JP9.39, JP9.40, U1G$1.GNDANA, U1G$1.GND_1, U1G$1.GND_2, U1G$1.GND_3, U2.GND, U3.GND; no longer C32.2, U1B.GND_1, U1B.GND_2, U7.GND
- net I2C_SCL: now also JP5.2; no longer U1A.PA17/SERCOM1/PAD1/SS/SCL
- net I2C_SDA: now also JP4.2; no longer U1A.PA16/SERCOM1/PAD0/SDA/MISO
- net P_GOOD: now also JP2.2; no longer JP2.1, U1A.PA14
- net RESET: now also U1G$1.!RESET; no longer U1B.!RESET
- net SPI_MISO: now also JP6.2; no longer U1A.PA08/SERCOM0/PAD0/MISO/SDA/AIN8
- net SPI_MOSI: now also JP7.2; no longer U1A.PA10/SERCOM0/PAD2/MOSI/AIN10
- net SPI_SCK: now also JP8.2; no longer U1A.PA11/SERCOM0/PAD3/SCK/AIN11
- net SWCLK: now also R4.1, U1G$1.PA30/SWCLK; no longer U1B.PA30/SWCLK
- net SWDIO: now also U1G$1.PA31/SWDIO; no longer U1B.PA31/SWDIO
- net UART_RX: now also JP9.6, U1G$2.PA05; no longer U1A.PA23/SERCOM3/PAD1/SCL/UARTRX
- net UART_TX: now also JP9.5, U1G$2.PA04; no longer U1A.PA22/SERCOM3/PAD0/SDA/UARTTX
