File: Hardware/PS-001/PS-001 - Copy.brd (EAGLE design)
At the start: 39.4 x 39.4 mm, 116 parts, among them IC1 LM5050Q1MKX-1_NOPB, IC2 LM5050Q1MKX-1_NOPB, IC3 LM5050Q1MKX-1_NOPB, J1 10144517-042802LF, J2 10144518-041802LF, J3 10144517-042802LF, J4 10144518-041802LF, J6 2X5_0.05_SWD, Q1 FDD86369-F085, Q2 DMG6968UQ-7, Q3 DMG6968UQ-7, U2 MAX16935CAUES/V+, U3 MAX16935CAUES/V+, U4 INA186A2IDCKT, U5 INA2180A4IDGKR, U6 NCV8170AXV330T2G, U7 ATA6561-GAQW-N

Commit message: updates to ps-001
Parts:
- moved R25 21.6 mm to (25.0, 6.48)
- moved C28 21.6 mm to (30.3, 4.29)
- moved C44 21.6 mm to (23.9, 6.38)
- moved R10 21.6 mm to (27.6, 4.19)
- moved R11 21.6 mm to (28.8, 4.19)
- moved R24 21.6 mm to (26.0, 6.48)
- moved U5 16.0 mm to (28.2, 4.52), turned to 90 degrees
- moved R28 11.4 mm to (29.2, 15.0)
- moved C35 11.1 mm to (27.0, 14.7), turned to 180 degrees
- moved R29 10.5 mm to (9.86, 17.3), turned to 0 degrees
- moved C37 8.13 mm to (23.2, 4.45)
- moved C38 8.13 mm to (23.2, 1.52)
- moved C39 8.13 mm to (20.4, 1.52)
- moved R12 8.13 mm to (17.7, 4.70)
- moved R13 8.13 mm to (17.7, 3.68)
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Routing:
- net PGND: track 94.9 -> 139.8 mm, vias 31 -> 39
- net N$30: track 0.00 -> 44.4 mm, vias 0 -> 4
- net +5V_INT_VMON: track 0.00 -> 32.9 mm, vias 0 -> 1
- net +12V_VMON: track 0.00 -> 32.0 mm, vias 0 -> 1
- net +12V_INT_VMON: track 0.00 -> 29.2 mm, vias 0 -> 1
- net +5V_VMON: track 0.00 -> 26.2 mm, vias 0 -> 1
- net DETECT_A: track 0.00 -> 23.9 mm, vias 0 -> 1
- net DETECT_B: track 0.00 -> 23.5 mm, vias 0 -> 2
- net +12V_REG: track 0.00 -> 23.4 mm, vias 0 -> 6
- net +12V_IMON: track 30.7 -> 47.9 mm
- net +5V_IMON_SENSE_N: track 0.00 -> 17.0 mm, vias 0 -> 2
- net +5V_IMON_SENSE_P: track 0.00 -> 16.6 mm, vias 0 -> 2
- net +5V_REG: track 0.08 -> 14.1 mm, vias 0 -> 5
- net DGND: track 18.8 -> 32.3 mm, vias 7 -> 12
- net +V_BAT: track 15.0 -> 27.3 mm, vias 14 -> 16
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- added copper zone on layer 1, net +12V_REG
- added copper zone on layer 16, net +12V_REG
- added copper zone on layer 16, net +5V_REG
- added copper zone on layer 16, net N$12
